Commit message: Rename/cleanup URDF stuff for f1tenth car

File: Simulator/f1_10_car_sim/urdf/racecar_gen.xacro (robot description, xacro)
@@ -1,5 +1,6 @@
 <?xml version="1.0"?>
-<robot name="racecar" xmlns:xacro="http://www.ros.org/wiki/xacro">
-  <xacro:include filename="$(find racecar_description)/urdf/macros.xacro" />
+<robot xmlns:xacro="http://www.ros.org/wiki/xacro" name=''>
+<!--Load the parameters passed in from other launch files -->
+  <xacro:include filename="$(find racecar_description)/urdf/macros_gen.xacro" />
   <!-- Add chassis and it's inertia link -->
   <link name="base_link" />
@@ -7,5 +8,5 @@
     <visual>
       <xacro:chassis_geometry/>
-      <material name="red" />
+      <material name="green" />
     </visual>
   </link>
@@ -254,5 +255,5 @@
   </joint>
   <!-- Add the remaining xacros -->
-  <xacro:include filename="$(find racecar_description)/urdf/racecar.gazebo" />
-  <xacro:include filename="$(find racecar_description)/urdf/materials.xacro" />
+  <xacro:include filename="$(find racecar_description)/urdf/racecar_gen.gazebo" />
+  <xacro:include filename="$(find racecar_description)/urdf/materials_gen.xacro" />
 </robot>
