Commit message: Refactored f1tenth_sim runs in Gazebo (melodic)

File: Simulator/f1tenth_sim/urdf/macros_gen.xacro (robot description, xacro)
@@ -41,5 +41,5 @@
   <origin xyz="0 0 0" rpy="0 0 0" />
   <geometry>
-    <mesh filename="package://racecar_description/meshes/chassis.STL" />
+    <mesh filename="package://f1tenth_sim/meshes/chassis.STL" />
   </geometry>
 </xacro:macro>
@@ -47,5 +47,5 @@
   <origin xyz="0 0 0" rpy="0 0 0" />
   <geometry>
-    <mesh filename="package://racecar_description/meshes/left_rear_wheel.STL" />
+    <mesh filename="package://f1tenth_sim/meshes/left_rear_wheel.STL" />
   </geometry>
 </xacro:macro>
@@ -53,5 +53,5 @@
   <origin xyz="0 0 0" rpy="0 0 0" />
   <geometry>
-    <mesh filename="package://racecar_description/meshes/right_rear_wheel.STL" />
+    <mesh filename="package://f1tenth_sim/meshes/right_rear_wheel.STL" />
   </geometry>
 </xacro:macro>
@@ -59,5 +59,5 @@
   <origin xyz="0 0 0" rpy="0 0 0" />
   <geometry>
-    <mesh filename="package://racecar_description/meshes/left_front_wheel.STL" />
+    <mesh filename="package://f1tenth_sim/meshes/left_front_wheel.STL" />
   </geometry>
 </xacro:macro>
@@ -65,5 +65,5 @@
   <origin xyz="0 0 0" rpy="0 0 0" />
   <geometry>
-    <mesh filename="package://racecar_description/meshes/right_front_wheel.STL" />
+    <mesh filename="package://f1tenth_sim/meshes/right_front_wheel.STL" />
   </geometry>
 </xacro:macro>
@@ -71,5 +71,5 @@
   <origin xyz="0 0 0" rpy="0 0 0" />
   <geometry>
-    <mesh filename="package://racecar_description/meshes/left_steering_hinge.STL" />
+    <mesh filename="package://f1tenth_sim/meshes/left_steering_hinge.STL" />
   </geometry>
 </xacro:macro>
@@ -77,5 +77,5 @@
   <origin xyz="0 0 0" rpy="0 0 0" />
   <geometry>
-    <mesh filename="package://racecar_description/meshes/right_steering_hinge.STL" />
+    <mesh filename="package://f1tenth_sim/meshes/right_steering_hinge.STL" />
   </geometry>
 </xacro:macro>

File: Simulator/f1tenth_sim/urdf/racecar_gen.xacro (robot description, xacro)
@@ -2,5 +2,5 @@
 <robot xmlns:xacro="http://www.ros.org/wiki/xacro" name=''>
 <!--Load the parameters passed in from other launch files -->
-  <xacro:include filename="$(find racecar_description)/urdf/macros_gen.xacro" />
+  <xacro:include filename="$(find f1tenth_sim)/urdf/macros_gen.xacro" />
   <!-- Add chassis and it's inertia link -->
   <link name="base_link" />
@@ -160,5 +160,5 @@
       <origin xyz="0 0 0" rpy="0 0 0"/>
       <geometry>
-        <mesh filename="package://racecar_description/meshes/hokuyo.dae"/>
+        <mesh filename="package://f1tenth_sim/meshes/hokuyo.dae"/>
         <material name="grey" />
       </geometry>
@@ -255,5 +255,5 @@
   </joint>
   <!-- Add the remaining xacros -->
-  <xacro:include filename="$(find racecar_description)/urdf/racecar_gen.gazebo" />
-  <xacro:include filename="$(find racecar_description)/urdf/materials_gen.xacro" />
+  <xacro:include filename="$(find f1tenth_sim)/urdf/racecar_gen.gazebo" />
+  <xacro:include filename="$(find f1tenth_sim)/urdf/materials_gen.xacro" />
 </robot>
