Commit message: Fix file names, combine alc_msgs, use component skeleton for Camera_Node

File: Simulator/f1tenth_sim/urdf/racecar_gen.xacro (robot description, xacro)
@@ -12,4 +12,5 @@
   </link>
   <joint name="base_link_joint" type="fixed">
+    <!-- <pose>-4 2 -.5 0 0 -1.57</pose> -->
     <origin xyz="0 0 0.05" rpy="0 0 0" />
     <parent link="base_link" />
@@ -71,9 +72,9 @@
   <link name="left_steering_hinge">
     <inertial>
-      <xacro:steering_hinge_inertial_params />
-    </inertial>
-    <visual>
-      <xacro:left_steering_hinge_geometry />
-      <material name="grey" />
+      <xacro:steering_hinge_inertial_params/>
+    </inertial>
+    <visual>
+      <xacro:left_steering_hinge_geometry/>
+      <material name="grey"/>
     </visual>
   </link>
